Commit message: fuck it works

File: body.urdf (robot description, URDF)
Before this commit: robot robot, 5 links, 4 joints
Links:
- added link BackLowerLeg, mass 1; collision box size=0.2 0.2 1.0; visual box size=0.2 0.2 1.0
- added link FrontLowerLeg, mass 1; collision box size=0.2 0.2 1.0; visual box size=0.2 0.2 1.0
- added link LeftLowerLeg, mass 1; collision box size=0.2 0.2 1.0; visual box size=0.2 0.2 1.0
- added link RightLowerLeg, mass 1; collision box size=0.2 0.2 1.0; visual box size=0.2 0.2 1.0
Joints:
- added joint BackLeg_BackLowerLeg: type revolute, parent BackLeg, child BackLowerLeg, origin xyz=0 -1.0 0 rpy=0 0 0, axis 0 1 0, limit lower=-3.14159 upper=3.14159 effort=0.0 velocity=0.0
- added joint FrontLeg_FrontLowerLeg: type revolute, parent FrontLeg, child FrontLowerLeg, origin xyz=0 1.0 0 rpy=0 0 0, axis 0 1 0, limit lower=-3.14159 upper=3.14159 effort=0.0 velocity=0.0
- added joint LeftLeg_LeftLowerLeg: type revolute, parent LeftLeg, child LeftLowerLeg, origin xyz=-1.0 0 0 rpy=0 0 0, axis 0 1 0, limit lower=-3.14159 upper=3.14159 effort=0.0 velocity=0.0
- added joint RightLeg_RightLowerLeg: type revolute, parent RightLeg, child RightLowerLeg, origin xyz=1.0 0 0 rpy=0 0 0, axis 0 1 0, limit lower=-3.14159 upper=3.14159 effort=0.0 velocity=0.0

Commit message: update geometry

File: body.urdf (robot description, URDF)
Before this commit: robot robot, 9 links, 8 joints
Links:
- removed link BackLeg
- removed link BackLowerLeg
- removed link FrontLeg
- removed link FrontLowerLeg
- removed link LeftLeg
- removed link LeftLowerLeg
- removed link RightLeg
- removed link RightLowerLeg
- added link BackLeftLeg, mass 1; collision box size=0.2 1.0 0.2; visual box size=0.2 1.0 0.2
- added link BackLeftLowerLeg, mass 1; collision box size=0.2 0.2 1.0; visual box size=0.2 0.2 1.0
- added link BackRightLeg, mass 1; collision box size=0.2 1.0 0.2; visual box size=0.2 1.0 0.2
- added link BackRightLowerLeg, mass 1; collision box size=0.2 0.2 1.0; visual box size=0.2 0.2 1.0
- added link FrontLeftLeg, mass 1; collision box size=0.2 1.0 0.2; visual box size=0.2 1.0 0.2
- added link FrontLeftLowerLeg, mass 1; collision box size=0.2 0.2 1.0; visual box size=0.2 0.2 1.0
- added link FrontRightLeg, mass 1; collision box size=0.2 1.0 0.2; visual box size=0.2 1.0 0.2
- added link FrontRightLowerLeg, mass 1; collision box size=0.2 0.2 1.0; visual box size=0.2 0.2 1.0
- added link MiddleLeftLeg, mass 1; collision box size=0.2 1.0 0.2; visual box size=0.2 1.0 0.2
- added link MiddleLeftLowerLeg, mass 1; collision box size=0.2 0.2 1.0; visual box size=0.2 0.2 1.0
- added link MiddleRightLeg, mass 1; collision box size=0.2 1.0 0.2; visual box size=0.2 1.0 0.2
- added link MiddleRightLowerLeg, mass 1; collision box size=0.2 0.2 1.0; visual box size=0.2 0.2 1.0
Joints:
- removed joint BackLeg_BackLowerLeg
- removed joint FrontLeg_FrontLowerLeg
- removed joint LeftLeg_LeftLowerLeg
- removed joint RightLeg_RightLowerLeg
- removed joint Torso_BackLeg
- removed joint Torso_FrontLeg
- removed joint Torso_LeftLeg
- removed joint Torso_RightLeg
- added joint BackLeftLeg_BackLeftLowerLeg: type revolute, parent BackLeftLeg, child BackLeftLowerLeg, origin xyz=0 1.0 0 rpy=0 0 0, axis 0 1 0, limit lower=-3.14159 upper=3.14159 effort=0.0 velocity=0.0
- added joint BackRightLeg_BackRightLowerLeg: type revolute, parent BackRightLeg, child BackRightLowerLeg, origin xyz=0 -1.0 0 rpy=0 0 0, axis 0 1 0, limit lower=-3.14159 upper=3.14159 effort=0.0 velocity=0.0
- added joint FrontLeftLeg_FrontLeftLowerLeg: type revolute, parent FrontLeftLeg, child FrontLeftLowerLeg, origin xyz=0 1.0 0 rpy=0 0 0, axis 0 1 0, limit lower=-3.14159 upper=3.14159 effort=0.0 velocity=0.0
- added joint FrontRightLeg_FrontRightLowerLeg: type revolute, parent FrontRightLeg, child FrontRightLowerLeg, origin xyz=0 -1.0 0 rpy=0 0 0, axis 0 1 0, limit lower=-3.14159 upper=3.14159 effort=0.0 velocity=0.0
- added joint MiddleLeftLeg_MiddleLeftLowerLeg: type revolute, parent MiddleLeftLeg, child MiddleLeftLowerLeg, origin xyz=0 1.0 0 rpy=0 0 0, axis 0 1 0, limit lower=-3.14159 upper=3.14159 effort=0.0 velocity=0.0
- added joint MiddleRightLeg_MiddleRightLowerLeg: type revolute, parent MiddleRightLeg, child MiddleRightLowerLeg, origin xyz=0 -1.0 0 rpy=0 0 0, axis 0 1 0, limit lower=-3.14159 upper=3.14159 effort=0.0 velocity=0.0
- added joint Torso_BackLeftLeg: type revolute, parent Torso, child BackLeftLeg, origin xyz=-0.5 0.5 1 rpy=0 0 0, axis 0 1 0, limit lower=-3.14159 upper=3.14159 effort=0.0 velocity=0.0
- added joint Torso_BackRightLeg: type revolute, parent Torso, child BackRightLeg, origin xyz=-0.5 -0.5 1 rpy=0 0 0, axis 0 1 0, limit lower=-3.14159 upper=3.14159 effort=0.0 velocity=0.0
- added joint Torso_FrontLeftLeg: type revolute, parent Torso, child FrontLeftLeg, origin xyz=0.5 0.5 1 rpy=0 0 0, axis 0 1 0, limit lower=-3.14159 upper=3.14159 effort=0.0 velocity=0.0
- added joint Torso_FrontRightLeg: type revolute, parent Torso, child FrontRightLeg, origin xyz=0.5 -0.5 1 rpy=0 0 0, axis 0 1 0, limit lower=-3.14159 upper=3.14159 effort=0.0 velocity=0.0
- added joint Torso_MiddleLeftLeg: type revolute, parent Torso, child MiddleLeftLeg, origin xyz=0 0.5 1 rpy=0 0 0, axis 0 1 0, limit lower=-3.14159 upper=3.14159 effort=0.0 velocity=0.0
- added joint Torso_MiddleRightLeg: type revolute, parent Torso, child MiddleRightLeg, origin xyz=0 -0.5 1 rpy=0 0 0, axis 0 1 0, limit lower=-3.14159 upper=3.14159 effort=0.0 velocity=0.0

Commit message: analyze3 woot

File: body.urdf (robot description, URDF)
Before this commit: robot robot, 13 links, 12 joints
Links:
- removed link BackLeftLeg
- removed link BackLeftLowerLeg
- removed link BackRightLeg
- removed link BackRightLowerLeg
- removed link FrontLeftLeg
- removed link FrontLeftLowerLeg
- removed link FrontRightLeg
- removed link FrontRightLowerLeg
- removed link MiddleLeftLeg
- removed link MiddleLeftLowerLeg
- removed link MiddleRightLeg
- removed link MiddleRightLowerLeg
- added link BackLeg, mass 1; collision box size=0.2 1 0.2; visual box size=0.2 1 0.2
- added link BackLowerLeg, mass 1; collision box size=0.2 0.2 1.0; visual box size=0.2 0.2 1.0
- added link FrontLeg, mass 1; collision box size=0.2 1 0.2; visual box size=0.2 1 0.2
- added link FrontLowerLeg, mass 1; collision box size=0.2 0.2 1.0; visual box size=0.2 0.2 1.0
- added link LeftLeg, mass 1; collision box size=1 0.2 0.2; visual box size=1 0.2 0.2
- added link LeftLowerLeg, mass 1; collision box size=0.2 0.2 1.0; visual box size=0.2 0.2 1.0
- added link RightLeg, mass 1; collision box size=1 0.2 0.2; visual box size=1 0.2 0.2
- added link RightLowerLeg, mass 1; collision box size=0.2 0.2 1.0; visual box size=0.2 0.2 1.0
Joints:
- removed joint BackLeftLeg_BackLeftLowerLeg
- removed joint BackRightLeg_BackRightLowerLeg
- removed joint FrontLeftLeg_FrontLeftLowerLeg
- removed joint FrontRightLeg_FrontRightLowerLeg
- removed joint MiddleLeftLeg_MiddleLeftLowerLeg
- removed joint MiddleRightLeg_MiddleRightLowerLeg
- removed joint Torso_BackLeftLeg
- removed joint Torso_BackRightLeg
- removed joint Torso_FrontLeftLeg
- removed joint Torso_FrontRightLeg
- removed joint Torso_MiddleLeftLeg
- removed joint Torso_MiddleRightLeg
- added joint BackLeg_BackLowerLeg: type revolute, parent BackLeg, child BackLowerLeg, origin xyz=0 -1.0 0 rpy=0 0 0, axis 0 1 0, limit lower=-3.14159 upper=3.14159 effort=0.0 velocity=0.0
- added joint FrontLeg_FrontLowerLeg: type revolute, parent FrontLeg, child FrontLowerLeg, origin xyz=0 1.0 0 rpy=0 0 0, axis 0 1 0, limit lower=-3.14159 upper=3.14159 effort=0.0 velocity=0.0
- added joint LeftLeg_LeftLowerLeg: type revolute, parent LeftLeg, child LeftLowerLeg, origin xyz=-1.0 0 0 rpy=0 0 0, axis 0 1 0, limit lower=-3.14159 upper=3.14159 effort=0.0 velocity=0.0
- added joint RightLeg_RightLowerLeg: type revolute, parent RightLeg, child RightLowerLeg, origin xyz=1.0 0 0 rpy=0 0 0, axis 0 1 0, limit lower=-3.14159 upper=3.14159 effort=0.0 velocity=0.0
- added joint Torso_BackLeg: type revolute, parent Torso, child BackLeg, origin xyz=0 -0.5 1 rpy=0 0 0, axis 0 1 0, limit lower=-3.14159 upper=3.14159 effort=0.0 velocity=0.0
- added joint Torso_FrontLeg: type revolute, parent Torso, child FrontLeg, origin xyz=0 0.5 1 rpy=0 0 0, axis 0 1 0, limit lower=-3.14159 upper=3.14159 effort=0.0 velocity=0.0
- added joint Torso_LeftLeg: type revolute, parent Torso, child LeftLeg, origin xyz=-0.5 0 1 rpy=0 0 0, axis 0 1 0, limit lower=-3.14159 upper=3.14159 effort=0.0 velocity=0.0
- added joint Torso_RightLeg: type revolute, parent Torso, child RightLeg, origin xyz=0.5 0 1 rpy=0 0 0, axis 0 1 0, limit lower=-3.14159 upper=3.14159 effort=0.0 velocity=0.0
